File: pcb/halfboard.sch (KiCad schematic (older format))
At the start: 54 parts, among them SW1 SW_PUSH, SW10 SW_PUSH, SW11 SW_PUSH, SW12 SW_PUSH, SW13 SW_PUSH, SW14 SW_PUSH, SW15 SW_PUSH, SW16 SW_PUSH, SW17 SW_PUSH, SW18 SW_PUSH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

Commit message: finish pcb using new schematics
Parts:
- BAT1: symbol Device:Battery -> halfboard-rescue:Battery-Device
- D1, D10, D11, D12, D13, D14, D15, D16, D17, D18, D19, D2, D20, D21, D22, D23, D24, D3, D4, D5, D6, D7, D8, D9: symbol Diode:1N4148W -> halfboard-rescue:1N4148W-Diode
- PWR_SW1, PWR_SW2, RESET1, RESET2: symbol Switch:SW_SPST -> halfboard-rescue:SW_SPST-Switch
- SW1, SW10, SW11, SW12, SW13, SW14, SW15, SW16, SW17, SW18, SW19, SW2, SW20, SW21, SW22, SW23, SW24, SW3, SW4, SW5, SW6, SW7, SW8, SW9: symbol sw_withled:SWITCH -> halfboard-rescue:SWITCH-sw_withled
- U1: symbol keebio:ProMicro -> halfboard-rescue:ProMicro-keebio
Connections:
- net col0: now also U1.20 (A3/PF4); no longer U1.9 (6/PD7)
- net col1: now also U1.19 (A2/PF5); no longer U1.11 (8/PB4)
- net col2: now also U1.18 (A1/PF6); no longer U1.12 (9/PB5)
- net col3: now also U1.17 (A0/PF7); no longer U1.20 (A3/PF4)
- net col4: now also U1.16 (15/PB1); no longer U1.19 (A2/PF5)
- net col5: now also U1.15 (14/PB3); no longer U1.18 (A1/PF6)
- net VCC: no longer names the net of U1.21 (VCC)
- no-connect marks 3 -> 9
Changed lines of the file:
@@
 encoding utf-8
 Sheet 1 1
-Title "REVIUNG41"
+Title "HALFBOARD"
 Date "2020-01-06"
 Rev "1.2"
@@
 $EndDescr
 $Comp
-L keebio:ProMicro U1
+L halfboard-rescue:ProMicro-keebio U1
 U 1 1 5DCBB133
 P 1800 2000
@@
 $EndComp
 $Comp
-L power:GND #PWR03
+L halfboard-rescue:GND-power #PWR03
 U 1 1 5DCBC44C
 P 2500 1550
@@
 	0    -1   -1   0
 $EndComp
-$Comp
-L power:VCC #PWR05
-U 1 1 5DCBC5E3
-P 2500 1750
-F 0 "#PWR05" H 2500 1600 50  0001 C CNN
-F 1 "VCC" V 2517 1878 50  0000 L CNN
-F 2 "" H 2500 1750 50  0001 C CNN
-F 3 "" H 2500 1750 50  0001 C CNN
-	1    2500 1750
-	0    1    1    0
-$EndComp
 Wire Wire Line
 	1100 1650 1050 1650
 $Comp
-L power:GND #PWR04
+L halfboard-rescue:GND-power #PWR04
 U 1 1 5DCBCA52
 P 1000 1650
@@
 	1050 1650 1000 1650
 $Comp
-L Diode:1N4148W D4
+L halfboard-rescue:1N4148W-Diode D4
 U 1 1 5DCC1C97
 P 6900 1500
@@
 $EndComp
 $Comp
-L sw_withled:SWITCH SW4
+L halfboard-rescue:SWITCH-sw_withled SW4
 U 1 1 5DCC1C91
 P 6600 1350
@@
 $EndComp
 $Comp
-L Diode:1N4148W D3
+L halfboard-rescue:1N4148W-Diode D3
 U 1 1 5DCC1C8B
 P 5900 1500
@@
 $EndComp
 $Comp
-L sw_withled:SWITCH SW3
+L halfboard-rescue:SWITCH-sw_withled SW3
 U 1 1 5DCC1C85
 P 5600 1350
@@
 $EndComp
 $Comp
-L Diode:1N4148W D2
+L halfboard-rescue:1N4148W-Diode D2
 U 1 1 5DCBF1A2
 P 4900 1500
@@
 $EndComp
 $Comp
-L sw_withled:SWITCH SW2
+L halfboard-rescue:SWITCH-sw_withled SW2
 U 1 1 5DCBF19C
 P 4600 1350
@@
 $EndComp
 $Comp
-L Diode:1N4148W D1
+L halfboard-rescue:1N4148W-Diode D1
 U 1 1 5DCBD469
 P 3900 1500
@@
 $EndComp
 $Comp
-L sw_withled:SWITCH SW1
+L halfboard-rescue:SWITCH-sw_withled SW1
 U 1 1 5DCBD08B
 P 3600 1350
@@
 $EndComp
 $Comp
-L sw_withled:SWITCH SW5
+L halfboard-rescue:SWITCH-sw_withled SW5
 U 1 1 5DCC4CE7
 P 7600 1350
@@
 $EndComp
 $Comp
-L Diode:1N4148W D5
+L halfboard-rescue:1N4148W-Diode D5
 U 1 1 5DCC4CED
 P 7900 1500
@@
 $EndComp
 $Comp
-L sw_withled:SWITCH SW6
+L halfboard-rescue:SWITCH-sw_withled SW6
 U 1 1 5DCC4CF3
 P 8600 1350
@@
 $EndComp
 $Comp
-L Diode:1N4148W D6
+L halfboard-rescue:1N4148W-Diode D6
 U 1 1 5DCC4CF9
 P 8900 1500
@@
 $EndComp
 $Comp
-L Diode:1N4148W D10
+L halfboard-rescue:1N4148W-Diode D10
 U 1 1 5DCCCAB6
 P 6900 2150
@@
 $EndComp
 $Comp
-L sw_withled:SWITCH SW10
+L halfboard-rescue:SWITCH-sw_withled SW10
 U 1 1 5DCCCABC
 P 6600 2000
@@
 $EndComp
 $Comp
-L Diode:1N4148W D9
+L halfboard-rescue:1N4148W-Diode D9
 U 1 1 5DCCCAC2
 P 5900 2150
@@
 $EndComp
 $Comp
-L sw_withled:SWITCH SW9
+L halfboard-rescue:SWITCH-sw_withled SW9
 U 1 1 5DCCCAC8
 P 5600 2000
@@
 $EndComp
 $Comp
-L Diode:1N4148W D8
+L halfboard-rescue:1N4148W-Diode D8
 U 1 1 5DCCCACE
 P 4900 2150
@@
 $EndComp
 $Comp
-L sw_withled:SWITCH SW8
+L halfboard-rescue:SWITCH-sw_withled SW8
 U 1 1 5DCCCAD4
 P 4600 2000
@@
 $EndComp
 $Comp
-L Diode:1N4148W D7
+L halfboard-rescue:1N4148W-Diode D7
 U 1 1 5DCCCADA
 P 3900 2150
@@
 $EndComp
 $Comp
-L sw_withled:SWITCH SW7
+L halfboard-rescue:SWITCH-sw_withled SW7
 U 1 1 5DCCCAE0
 P 3600 2000
@@
 $EndComp
 $Comp
-L sw_withled:SWITCH SW11
+L halfboard-rescue:SWITCH-sw_withled SW11
 U 1 1 5DCCCAE6
 P 7600 2000
@@
 $EndComp
 $Comp
-L Diode:1N4148W D11
+L halfboard-rescue:1N4148W-Diode D11
 U 1 1 5DCCCAEC
 P 7900 2150
@@
 $EndComp
 $Comp
-L sw_withled:SWITCH SW12
+L halfboard-rescue:SWITCH-sw_withled SW12
 U 1 1 5DCCCAF2
 P 8600 2000
@@
 $EndComp
 $Comp
-L Diode:1N4148W D12
+L halfboard-rescue:1N4148W-Diode D12
 U 1 1 5DCCCAF8
 P 8900 2150
@@
 $EndComp
 $Comp
-L Diode:1N4148W D16
+L halfboard-rescue:1N4148W-Diode D16
 U 1 1 5DCD2B3B
 P 6900 2800
@@
 $EndComp
 $Comp
-L sw_withled:SWITCH SW16
+L halfboard-rescue:SWITCH-sw_withled SW16
 U 1 1 5DCD2B41
 P 6600 2650
@@
 $EndComp
 $Comp
-L Diode:1N4148W D15
+L halfboard-rescue:1N4148W-Diode D15
 U 1 1 5DCD2B47
 P 5900 2800
@@
 $EndComp
 $Comp
-L sw_withled:SWITCH SW15
+L halfboard-rescue:SWITCH-sw_withled SW15
 U 1 1 5DCD2B4D
 P 5600 2650
@@
 $EndComp
 $Comp
-L Diode:1N4148W D14
+L halfboard-rescue:1N4148W-Diode D14
 U 1 1 5DCD2B53
 P 4900 2800
@@
 $EndComp
 $Comp
-L sw_withled:SWITCH SW14
+L halfboard-rescue:SWITCH-sw_withled SW14
 U 1 1 5DCD2B59
 P 4600 2650
@@
 $EndComp
 $Comp
-L Diode:1N4148W D13
+L halfboard-rescue:1N4148W-Diode D13
 U 1 1 5DCD2B5F
 P 3900 2800
@@
 $EndComp
 $Comp
-L sw_withled:SWITCH SW13
+L halfboard-rescue:SWITCH-sw_withled SW13
 U 1 1 5DCD2B65
 P 3600 2650
@@
 $EndComp
 $Comp
-L sw_withled:SWITCH SW17
+L halfboard-rescue:SWITCH-sw_withled SW17
 U 1 1 5DCD2B6B
 P 7600 2650
@@
 $EndComp
 $Comp
-L Diode:1N4148W D17
+L halfboard-rescue:1N4148W-Diode D17
 U 1 1 5DCD2B71
 P 7900 2800
@@
 $EndComp
 $Comp
-L sw_withled:SWITCH SW18
+L halfboard-rescue:SWITCH-sw_withled SW18
 U 1 1 5DCD2B77
 P 8600 2650
@@
 $EndComp
 $Comp
-L Diode:1N4148W D18
+L halfboard-rescue:1N4148W-Diode D18
 U 1 1 5DCD2B7D
 P 8900 2800
@@
 $EndComp
 $Comp
-L Diode:1N4148W D22
+L halfboard-rescue:1N4148W-Diode D22
 U 1 1 5DCD8200
 P 6900 3450
@@
 $EndComp
 $Comp
-L sw_withled:SWITCH SW22
+L halfboard-rescue:SWITCH-sw_withled SW22
 U 1 1 5DCD8206
 P 6600 3300
@@
 $EndComp
 $Comp
-L Diode:1N4148W D21
+L halfboard-rescue:1N4148W-Diode D21
 U 1 1 5DCD820C
 P 5900 3450
@@
 $EndComp
 $Comp
-L sw_withled:SWITCH SW21
+L halfboard-rescue:SWITCH-sw_withled SW21
 U 1 1 5DCD8212
 P 5600 3300
@@
 $EndComp
 $Comp
-L Diode:1N4148W D20
+L halfboard-rescue:1N4148W-Diode D20
 U 1 1 5DCD8218
 P 4900 3450
@@
 $EndComp
 $Comp
-L sw_withled:SWITCH SW20
+L halfboard-rescue:SWITCH-sw_withled SW20
 U 1 1 5DCD821E
 P 4600 3300
@@
 $EndComp
 $Comp
-L Diode:1N4148W D19
+L halfboard-rescue:1N4148W-Diode D19
 U 1 1 5DCD8224
 P 3900 3450
@@
 $EndComp
 $Comp
-L sw_withled:SWITCH SW19
+L halfboard-rescue:SWITCH-sw_withled SW19
 U 1 1 5DCD822A
 P 3600 3300
@@
 $EndComp
 $Comp
-L sw_withled:SWITCH SW23
+L halfboard-rescue:SWITCH-sw_withled SW23
 U 1 1 5DCD8230
 P 7600 3300
@@
 $EndComp
 $Comp
-L Diode:1N4148W D23
+L halfboard-rescue:1N4148W-Diode D23
 U 1 1 5DCD8236
 P 7900 3450
@@
 $EndComp
 $Comp
-L sw_withled:SWITCH SW24
+L halfboard-rescue:SWITCH-sw_withled SW24
 U 1 1 5DCD823C
 P 8600 3300
@@
 $EndComp
 $Comp
-L Diode:1N4148W D24
+L halfboard-rescue:1N4148W-Diode D24
 U 1 1 5DCD8242
 P 8900 3450
@@
 Connection ~ 7900 3600
 $Comp
-L power:GND #PWR08
+L halfboard-rescue:GND-power #PWR08
 U 1 1 5DD425AD
 P 2100 3350
@@
 Text GLabel 1100 2150 0    50   Input ~ 0
 row3
-Text GLabel 1100 2250 0    50   Input ~ 0
-col0
-Text GLabel 1100 2450 0    50   Input ~ 0
-col1
-Text GLabel 1100 2550 0    50   Input ~ 0
-col2
+Text GLabel 2500 2250 2    50   Input ~ 0
+col4
+Text GLabel 2500 2350 2    50   Input ~ 0
+col5
 Text GLabel 2500 1650 2    50   Input ~ 0
 reset
 Text GLabel 2500 1850 2    50   Input ~ 0
-col3
+col0
 Text GLabel 2500 1950 2    50   Input ~ 0
-col4
+col1
 Text GLabel 2500 2050 2    50   Input ~ 0
-col5
+col2
 Text GLabel 3200 1650 0    50   Input ~ 0
 row0
@@
 reset
 $Comp
-L Switch:SW_SPST RESET1
+L halfboard-rescue:SW_SPST-Switch RESET1
 U 1 1 5DD41146
 P 1800 3350
@@
 row0
 $Comp
-L Switch:SW_SPST PWR_SW1
+L halfboard-rescue:SW_SPST-Switch PWR_SW1
 U 1 1 602C7F72
 P 1500 3950
@@
 $EndComp
 $Comp
-L power:GND #PWR0101
+L halfboard-rescue:GND-power #PWR0101
 U 1 1 600F2961
 P 1250 3950
@@
 	1300 3950 1250 3950
 $Comp
-L Device:Battery BAT1
+L halfboard-rescue:Battery-Device BAT1
 U 1 1 60102ED1
 P 2100 3950
@@
 	2400 3950 2300 3950
 $Comp
-L power:GND #PWR?
+L halfboard-rescue:GND-power #PWR?
 U 1 1 60254313
 P 2100 3000
@@
 reset
 $Comp
-L Switch:SW_SPST RESET2
+L halfboard-rescue:SW_SPST-Switch RESET2
 U 1 1 6025431A
 P 1800 3000
@@
 	2000 3000 2100 3000
 $Comp
-L Switch:SW_SPST PWR_SW2
+L halfboard-rescue:SW_SPST-Switch PWR_SW2
 U 1 1 6025A6E4
 P 1500 4350
@@
 $EndComp
 $Comp
-L power:GND #PWR?
+L halfboard-rescue:GND-power #PWR?
 U 1 1 6025A6EA
 P 1250 4350
@@
 Wire Wire Line
 	1900 3950 1900 4350
+NoConn ~ 2500 1750
+Text GLabel 2500 2150 2    50   Input ~ 0
+col3
+NoConn ~ 2500 2450
+NoConn ~ 2500 2550
+NoConn ~ 1100 2250
+NoConn ~ 1100 2450
+NoConn ~ 1100 2550
 $EndSCHEMATC

Commit message: add ground plane
Parts:
- BAT1: symbol halfboard-rescue:Battery-Device -> halfboard:Battery-Device
- D1, D10, D11, D12, D13, D14, D15, D16, D17, D18, D19, D2, D20, D21, D22, D23, D24, D3, D4, D5, D6, D7, D8, D9: symbol halfboard-rescue:1N4148W-Diode -> halfboard:1N4148W-Diode
- PWR_SW1, PWR_SW2, RESET1, RESET2: symbol halfboard-rescue:SW_SPST-Switch -> halfboard:SW_SPST-Switch
- SW1, SW10, SW11, SW12, SW13, SW14, SW15, SW16, SW17, SW18, SW19, SW2, SW20, SW21, SW22, SW23, SW24, SW3, SW4, SW5, SW6, SW7, SW8, SW9: symbol halfboard-rescue:SWITCH-sw_withled -> halfboard:SWITCH-sw_withled
- U1: symbol halfboard-rescue:ProMicro-keebio -> halfboard:ProMicro-keebio
Changed lines of the file:
@@
 $EndDescr
 $Comp
-L halfboard-rescue:ProMicro-keebio U1
+L halfboard:ProMicro-keebio U1
 U 1 1 5DCBB133
 P 1800 2000
@@
 $EndComp
 $Comp
-L halfboard-rescue:GND-power #PWR03
+L halfboard:GND-power #PWR03
 U 1 1 5DCBC44C
 P 2500 1550
@@
 	1100 1650 1050 1650
 $Comp
-L halfboard-rescue:GND-power #PWR04
+L halfboard:GND-power #PWR04
 U 1 1 5DCBCA52
 P 1000 1650
@@
 	1050 1650 1000 1650
 $Comp
-L halfboard-rescue:1N4148W-Diode D4
+L halfboard:1N4148W-Diode D4
 U 1 1 5DCC1C97
 P 6900 1500
@@
 $EndComp
 $Comp
-L halfboard-rescue:SWITCH-sw_withled SW4
+L halfboard:SWITCH-sw_withled SW4
 U 1 1 5DCC1C91
 P 6600 1350
@@
 $EndComp
 $Comp
-L halfboard-rescue:1N4148W-Diode D3
+L halfboard:1N4148W-Diode D3
 U 1 1 5DCC1C8B
 P 5900 1500
@@
 $EndComp
 $Comp
-L halfboard-rescue:SWITCH-sw_withled SW3
+L halfboard:SWITCH-sw_withled SW3
 U 1 1 5DCC1C85
 P 5600 1350
@@
 $EndComp
 $Comp
-L halfboard-rescue:1N4148W-Diode D2
+L halfboard:1N4148W-Diode D2
 U 1 1 5DCBF1A2
 P 4900 1500
@@
 $EndComp
 $Comp
-L halfboard-rescue:SWITCH-sw_withled SW2
+L halfboard:SWITCH-sw_withled SW2
 U 1 1 5DCBF19C
 P 4600 1350
@@
 $EndComp
 $Comp
-L halfboard-rescue:1N4148W-Diode D1
+L halfboard:1N4148W-Diode D1
 U 1 1 5DCBD469
 P 3900 1500
@@
 $EndComp
 $Comp
-L halfboard-rescue:SWITCH-sw_withled SW1
+L halfboard:SWITCH-sw_withled SW1
 U 1 1 5DCBD08B
 P 3600 1350
@@
 $EndComp
 $Comp
-L halfboard-rescue:SWITCH-sw_withled SW5
+L halfboard:SWITCH-sw_withled SW5
 U 1 1 5DCC4CE7
 P 7600 1350
@@
 $EndComp
 $Comp
-L halfboard-rescue:1N4148W-Diode D5
+L halfboard:1N4148W-Diode D5
 U 1 1 5DCC4CED
 P 7900 1500
@@
 $EndComp
 $Comp
-L halfboard-rescue:SWITCH-sw_withled SW6
+L halfboard:SWITCH-sw_withled SW6
 U 1 1 5DCC4CF3
 P 8600 1350
@@
 $EndComp
 $Comp
-L halfboard-rescue:1N4148W-Diode D6
+L halfboard:1N4148W-Diode D6
 U 1 1 5DCC4CF9
 P 8900 1500
@@
 $EndComp
 $Comp
-L halfboard-rescue:1N4148W-Diode D10
+L halfboard:1N4148W-Diode D10
 U 1 1 5DCCCAB6
 P 6900 2150
@@
 $EndComp
 $Comp
-L halfboard-rescue:SWITCH-sw_withled SW10
+L halfboard:SWITCH-sw_withled SW10
 U 1 1 5DCCCABC
 P 6600 2000
@@
 $EndComp
 $Comp
-L halfboard-rescue:1N4148W-Diode D9
+L halfboard:1N4148W-Diode D9
 U 1 1 5DCCCAC2
 P 5900 2150
@@
 $EndComp
 $Comp
-L halfboard-rescue:SWITCH-sw_withled SW9
+L halfboard:SWITCH-sw_withled SW9
 U 1 1 5DCCCAC8
 P 5600 2000
@@
 $EndComp
 $Comp
-L halfboard-rescue:1N4148W-Diode D8
+L halfboard:1N4148W-Diode D8
 U 1 1 5DCCCACE
 P 4900 2150
@@
 $EndComp
 $Comp
-L halfboard-rescue:SWITCH-sw_withled SW8
+L halfboard:SWITCH-sw_withled SW8
 U 1 1 5DCCCAD4
 P 4600 2000
@@
 $EndComp
 $Comp
-L halfboard-rescue:1N4148W-Diode D7
+L halfboard:1N4148W-Diode D7
 U 1 1 5DCCCADA
 P 3900 2150
@@
 $EndComp
 $Comp
-L halfboard-rescue:SWITCH-sw_withled SW7
+L halfboard:SWITCH-sw_withled SW7
 U 1 1 5DCCCAE0
 P 3600 2000
@@
 $EndComp
 $Comp
-L halfboard-rescue:SWITCH-sw_withled SW11
+L halfboard:SWITCH-sw_withled SW11
 U 1 1 5DCCCAE6
 P 7600 2000
@@
 $EndComp
 $Comp
-L halfboard-rescue:1N4148W-Diode D11
+L halfboard:1N4148W-Diode D11
 U 1 1 5DCCCAEC
 P 7900 2150
@@
 $EndComp
 $Comp
-L halfboard-rescue:SWITCH-sw_withled SW12
+L halfboard:SWITCH-sw_withled SW12
 U 1 1 5DCCCAF2
 P 8600 2000
@@
 $EndComp
 $Comp
-L halfboard-rescue:1N4148W-Diode D12
+L halfboard:1N4148W-Diode D12
 U 1 1 5DCCCAF8
 P 8900 2150
@@
 $EndComp
 $Comp
-L halfboard-rescue:1N4148W-Diode D16
+L halfboard:1N4148W-Diode D16
 U 1 1 5DCD2B3B
 P 6900 2800
@@
 $EndComp
 $Comp
-L halfboard-rescue:SWITCH-sw_withled SW16
+L halfboard:SWITCH-sw_withled SW16
 U 1 1 5DCD2B41
 P 6600 2650
@@
 $EndComp
 $Comp
-L halfboard-rescue:1N4148W-Diode D15
+L halfboard:1N4148W-Diode D15
 U 1 1 5DCD2B47
 P 5900 2800
@@
 $EndComp
 $Comp
-L halfboard-rescue:SWITCH-sw_withled SW15
+L halfboard:SWITCH-sw_withled SW15
 U 1 1 5DCD2B4D
 P 5600 2650
@@
 $EndComp
 $Comp
-L halfboard-rescue:1N4148W-Diode D14
+L halfboard:1N4148W-Diode D14
 U 1 1 5DCD2B53
 P 4900 2800
@@
 $EndComp
 $Comp
-L halfboard-rescue:SWITCH-sw_withled SW14
+L halfboard:SWITCH-sw_withled SW14
 U 1 1 5DCD2B59
 P 4600 2650
@@
 $EndComp
 $Comp
-L halfboard-rescue:1N4148W-Diode D13
+L halfboard:1N4148W-Diode D13
 U 1 1 5DCD2B5F
 P 3900 2800
@@
 $EndComp
 $Comp
-L halfboard-rescue:SWITCH-sw_withled SW13
+L halfboard:SWITCH-sw_withled SW13
 U 1 1 5DCD2B65
 P 3600 2650
@@
 $EndComp
 $Comp
-L halfboard-rescue:SWITCH-sw_withled SW17
+L halfboard:SWITCH-sw_withled SW17
 U 1 1 5DCD2B6B
 P 7600 2650
@@
 $EndComp
 $Comp
-L halfboard-rescue:1N4148W-Diode D17
+L halfboard:1N4148W-Diode D17
 U 1 1 5DCD2B71
 P 7900 2800
@@
 $EndComp
 $Comp
-L halfboard-rescue:SWITCH-sw_withled SW18
+L halfboard:SWITCH-sw_withled SW18
 U 1 1 5DCD2B77
 P 8600 2650
@@
 $EndComp
 $Comp
-L halfboard-rescue:1N4148W-Diode D18
+L halfboard:1N4148W-Diode D18
 U 1 1 5DCD2B7D
 P 8900 2800
@@
 $EndComp
 $Comp
-L halfboard-rescue:1N4148W-Diode D22
+L halfboard:1N4148W-Diode D22
 U 1 1 5DCD8200
 P 6900 3450
@@
 $EndComp
 $Comp
-L halfboard-rescue:SWITCH-sw_withled SW22
+L halfboard:SWITCH-sw_withled SW22
 U 1 1 5DCD8206
 P 6600 3300
@@
 $EndComp
 $Comp
-L halfboard-rescue:1N4148W-Diode D21
+L halfboard:1N4148W-Diode D21
 U 1 1 5DCD820C
 P 5900 3450
@@
 $EndComp
 $Comp
-L halfboard-rescue:SWITCH-sw_withled SW21
+L halfboard:SWITCH-sw_withled SW21
 U 1 1 5DCD8212
 P 5600 3300
@@
 $EndComp
 $Comp
-L halfboard-rescue:1N4148W-Diode D20
+L halfboard:1N4148W-Diode D20
 U 1 1 5DCD8218
 P 4900 3450
@@
 $EndComp
 $Comp
-L halfboard-rescue:SWITCH-sw_withled SW20
+L halfboard:SWITCH-sw_withled SW20
 U 1 1 5DCD821E
 P 4600 3300
@@
 $EndComp
 $Comp
-L halfboard-rescue:1N4148W-Diode D19
+L halfboard:1N4148W-Diode D19
 U 1 1 5DCD8224
 P 3900 3450
@@
 $EndComp
 $Comp
-L halfboard-rescue:SWITCH-sw_withled SW19
+L halfboard:SWITCH-sw_withled SW19
 U 1 1 5DCD822A
 P 3600 3300
@@
 $EndComp
 $Comp
-L halfboard-rescue:SWITCH-sw_withled SW23
+L halfboard:SWITCH-sw_withled SW23
 U 1 1 5DCD8230
 P 7600 3300
@@
 $EndComp
 $Comp
-L halfboard-rescue:1N4148W-Diode D23
+L halfboard:1N4148W-Diode D23
 U 1 1 5DCD8236
 P 7900 3450
@@
 $EndComp
 $Comp
-L halfboard-rescue:SWITCH-sw_withled SW24
+L halfboard:SWITCH-sw_withled SW24
 U 1 1 5DCD823C
 P 8600 3300
@@
 $EndComp
 $Comp
-L halfboard-rescue:1N4148W-Diode D24
+L halfboard:1N4148W-Diode D24
 U 1 1 5DCD8242
 P 8900 3450
@@
 Connection ~ 7900 3600
 $Comp
-L halfboard-rescue:GND-power #PWR08
+L halfboard:GND-power #PWR08
 U 1 1 5DD425AD
 P 2100 3350
@@
 reset
 $Comp
-L halfboard-rescue:SW_SPST-Switch RESET1
+L halfboard:SW_SPST-Switch RESET1
 U 1 1 5DD41146
 P 1800 3350
@@
 row0
 $Comp
-L halfboard-rescue:SW_SPST-Switch PWR_SW1
+L halfboard:SW_SPST-Switch PWR_SW1
 U 1 1 602C7F72
 P 1500 3950
@@
 $EndComp
 $Comp
-L halfboard-rescue:GND-power #PWR0101
+L halfboard:GND-power #PWR0101
 U 1 1 600F2961
 P 1250 3950
@@
 	1300 3950 1250 3950
 $Comp
-L halfboard-rescue:Battery-Device BAT1
+L halfboard:Battery-Device BAT1
 U 1 1 60102ED1
 P 2100 3950
@@
 	2400 3950 2300 3950
 $Comp
-L halfboard-rescue:GND-power #PWR?
+L halfboard:GND-power #PWR?
 U 1 1 60254313
 P 2100 3000
@@
 reset
 $Comp
-L halfboard-rescue:SW_SPST-Switch RESET2
+L halfboard:SW_SPST-Switch RESET2
 U 1 1 6025431A
 P 1800 3000
@@
 	2000 3000 2100 3000
 $Comp
-L halfboard-rescue:SW_SPST-Switch PWR_SW2
+L halfboard:SW_SPST-Switch PWR_SW2
 U 1 1 6025A6E4
 P 1500 4350
@@
 $EndComp
 $Comp
-L halfboard-rescue:GND-power #PWR?
+L halfboard:GND-power #PWR?
 U 1 1 6025A6EA
 P 1250 4350

Commit message: 5x4 layout instead of 6x4
Parts:
- removed D12, D18, D24, D6: 1N4148W, halfboard:Diode-dual, symbol halfboard:1N4148W-Diode
- removed PWR_SW2: SW_SPST, Button_Switch_SMD:SW_SPDT_PCM12, symbol halfboard:SW_SPST-Switch
- removed RESET1, RESET2: SW_PUSH, Button_Switch_SMD:SW_SPST_TL3342, symbol halfboard:SW_SPST-Switch
- removed SW12, SW18, SW24, SW6: SW_PUSH, halfboard:MX-ALPs-PG1350-LED-FLIP, symbol halfboard:SWITCH-sw_withled
- added D25, D26, D27, D28, D29: 1N4148W, halfboard:Diode-dual, symbol halfboard:1N4148W-Diode
- added SW25, SW26, SW27, SW28, SW29: SW_PUSH, halfboard:MX-ALPs-PG1350-LED-FLIP, symbol halfboard:SWITCH-sw_withled
Connections:
- net col0: now also SW25.1
- net col1: now also SW26.1
- net col2: now also SW27.1
- net col3: now also SW28.1
- net col4: now also SW29.1
- net row4: now reaches U1.9 (6/PD7)
- net row4: now also D25.1 (K), D26.1 (K), D27.1 (K), D28.1 (K), D29.1 (K)
- net col5: no longer names the net of U1.15 (14/PB3)
- new net: D28.2 (A), SW28.2
- new net: D27.2 (A), SW27.2
- new net: D26.2 (A), SW26.2
- new net: D25.2 (A), SW25.2
- new net: D29.2 (A), SW29.2
Other:
- moved on the sheet: BAT1, PWR_SW1
